File: HKIA_Tracker.kicad_pcb (KiCad board)
At the start: 4 copper layers, 85 parts, among them J1 Motor In, J2 SWD, J3 Conn_01x06, J4 Battery, J5 Conn_01x04, SW1 SW_Push, SW2 SW_Push, SW3 SW_Push, SW4 SW_Push, SW5 SW_Push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

Commit message: done
Parts:
- added H1: M3, MountingHole:MountingHole_3.2mm_M3_Pad, F.Cu at (145.0, 120.0)
- added H2: M3, MountingHole:MountingHole_3.2mm_M3_Pad, F.Cu at (105.0, 80.0)
- C17, C20, C24, J5, R20, R21, R22, R23, R24, SW4, SW5, U3: moved to B.Cu
- J1: footprint Connector_PinHeader_2.54mm:PinHeader_1x03_P2.54mm_Horizontal -> Connector_PinHeader_2.54mm:PinHeader_1x03_P2.54mm_Vertical
- J3: value Conn_01x06 -> NFC_ANT; footprint Connector_PinHeader_2.54mm:PinHeader_1x06_P2.54mm_Vertical -> Connector_PinHeader_2.54mm:PinHeader_1x02_P2.54mm_Vertical
- moved C25 80.9 mm to (138.3, 109.2), turned to 270 degrees
- moved C20 79.6 mm to (125.4, 101.7)
- moved C22 79.0 mm to (136.4, 109.4), turned to 270 degrees
- moved C17 77.8 mm to (128.2, 100.8), turned to 270 degrees
- moved SW4 77.1 mm to (141.9, 100.4)
- moved C18 77.1 mm to (133.7, 110.1), turned to 180 degrees
- moved R20 76.1 mm to (137.9, 99.9)
- moved R21 76.1 mm to (134.7, 99.9)
- moved L3 76.0 mm to (136.8, 105.7), turned to 0 degrees
- moved C24 75.8 mm to (125.6, 99.8)
- moved R27 75.4 mm to (133.7, 108.5), turned to 180 degrees
- moved C19 73.9 mm to (130.5, 110.1), turned to 180 degrees
- moved R28 72.2 mm to (130.5, 108.5), turned to 180 degrees
- moved U4 71.3 mm to (132.3, 105.7), turned to 0 degrees
- moved J2 68.8 mm to (137.3, 91.1)
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Connections:
- D7 pad 1: Net-(C7-Pad1) -> GND
- D7 pad 2: GND -> Net-(C7-Pad1)
- D7 pad 3: (no net) -> GND
- D7 pad 4: (no net) -> Net-(C7-Pad1)
- J1 pad 1: Net-(D1-Pad2) -> Net-(D5-Pad2)
- J1 pad 3: Net-(D5-Pad2) -> Net-(D1-Pad2)
- J3 pad 1: +3V3 -> Net-(J3-Pad1)
- J3 pad 2: /GPIO12 -> Net-(J3-Pad2)
- J4 pad MP: (no net) -> GND
- U1 pad 24: Net-(U1-Pad24) -> Net-(J3-Pad1)
- U1 pad 25: Net-(U1-Pad24) -> Net-(J3-Pad2)
- U1 pad 27: /GPIO12 -> Net-(U1-Pad27)
- U1 pad 28: /GPIO13 -> Net-(U1-Pad28)
- U1 pad 29: /GPIO14 -> Net-(U1-Pad29)
- U1 pad 30: /GPIO15 -> Net-(U1-Pad30)
Routing:
- net GND: track 0.00 -> 84.1 mm, vias 0 -> 99
- net /NRF_RX: track 0.00 -> 29.7 mm, vias 0 -> 1
- net /SWO: track 0.00 -> 22.4 mm
- net +3V3: track 0.00 -> 20.2 mm, vias 0 -> 24
- net +BATT: track 0.00 -> 19.7 mm, vias 0 -> 2
- net /nRST: track 0.00 -> 18.6 mm
- net /NRF_TX: track 0.00 -> 18.2 mm, vias 0 -> 1
- net /ESP_EN: track 0.00 -> 16.7 mm, vias 0 -> 2
- net /SWCLK: track 0.00 -> 16.2 mm
- net /SWDIO: track 0.00 -> 14.6 mm
- net Net-(R11-Pad1): track 0.00 -> 14.4 mm
- net /SDA: track 0.00 -> 12.8 mm, vias 0 -> 2
- net /SCL: track 0.00 -> 10.4 mm, vias 0 -> 2
- net Net-(R10-Pad2): track 0.00 -> 9.50 mm, vias 0 -> 3
- net /DRDY: track 0.00 -> 9.06 mm, vias 0 -> 2
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- added copper zone on B.Cu, net +3.3VP
- added copper zone on F.Cu, net +3.3VP
- added copper zone on In2.Cu, net +3.3VP
- added copper zone on F.Cu, net +3V3
- added copper zone on In2.Cu, net +3V3
- added copper zone on F.Cu, net +BATT
- added copper zone on F.Cu, net GND
- added copper zone on In1.Cu, net GND
- added copper zone on F.Cu, net Net-(C11-Pad1)
- added copper zone on F.Cu, net Net-(C14-Pad1)
- added copper zone on B.Cu, net Net-(C7-Pad1)
- added copper zone on F.Cu, net Net-(C7-Pad1)
- added copper zone on F.Cu, net Net-(D1-Pad1)
- added copper zone on F.Cu, net Net-(D1-Pad2)
- added copper zone on F.Cu, net Net-(D3-Pad2)
- added copper zone on B.Cu, net Net-(D5-Pad2)
- added copper zone on F.Cu, net Net-(D5-Pad2)
- added copper zone on F.Cu, net Net-(J4-Pad1)
- added copper zone on F.Cu, net Net-(L2-Pad2)
- added copper zone on F.Cu, net Net-(L3-Pad1)
- added copper zone on F.Cu, net VBUS
- added copper zone on In2.Cu, net VBUS
Other:
- board outline added: 50 x 50 mm
- board text added: "ALEX WONG"
- board text added: "BAT"
- board text added: "G"
- board text added: "HKUST ISD 2021 SPRING ISDN3002 TEAM AAJ TROLLEY TRACKER"
- board text added: "IO0"
- board text added: "NFC ANT"
- board text added: "P0.19"
- board text added: "P0.20"
- board text added: "P0.23"
- board text added: "P0.24"
- board text added: "PWR IN"
- board text added: "R"
- board text added: "RST"
- board text added: "SWD"
- board text added: "T"
- board text added: "V"
