File: HKIA_Tracker.sch (KiCad schematic (older format))
At the start: 85 parts, among them J1 Motor In, J2 SWD, J3 Conn_01x06, J4 Battery, J5 Conn_01x04, SW1 SW_Push, SW2 SW_Push, SW3 SW_Push, SW4 SW_Push, SW5 SW_Push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

Commit message: init placement
Connections:
- wire segments 247 -> 249
Other:
- moved on the sheet: D8, D9, R22, R23, R7, R8, SW5
Changed lines of the file:
@@
 L Switch:SW_Push SW5
 U 1 1 60DF4A9E
-P 10250 6450
-F 0 "SW5" V 10250 6598 50  0000 L CNN
-F 1 "SW_Push" V 10295 6598 50  0001 L CNN
-F 2 "Button_Switch_SMD:SW_SPST_CK_KXT3" H 10250 6650 50  0001 C CNN
-F 3 "~" H 10250 6650 50  0001 C CNN
-F 4 "C221821" V 10250 6450 50  0001 C CNN "LCSC"
-	1    10250 6450
-	0    1    1    0
+P 9900 6600
+F 0 "SW5" H 9900 6793 50  0000 C CNN
+F 1 "SW_Push" V 9945 6748 50  0001 L CNN
+F 2 "Button_Switch_SMD:SW_SPST_CK_KXT3" H 9900 6800 50  0001 C CNN
+F 3 "~" H 9900 6800 50  0001 C CNN
+F 4 "C221821" V 9900 6600 50  0001 C CNN "LCSC"
+	1    9900 6600
+	1    0    0    -1
 $EndComp
 $Comp
@@
 L Device:R R22
 U 1 1 60EF642A
-P 9850 5950
-F 0 "R22" V 9800 6150 50  0000 C CNN
-F 1 "10K" V 9900 5750 50  0000 C CNN
-F 2 "Resistor_SMD:R_0603_1608Metric" V 9780 5950 50  0001 C CNN
-F 3 "~" H 9850 5950 50  0001 C CNN
-F 4 "C98220" V 9850 5950 50  0001 C CNN "LCSC"
-	1    9850 5950
-	0    1    1    0
-$EndComp
-Wire Wire Line
-	9000 5950 9700 5950
+P 9900 5950
+F 0 "R22" V 9850 6150 50  0000 C CNN
+F 1 "10K" V 9950 5750 50  0000 C CNN
+F 2 "Resistor_SMD:R_0603_1608Metric" V 9830 5950 50  0001 C CNN
+F 3 "~" H 9900 5950 50  0001 C CNN
+F 4 "C98220" V 9900 5950 50  0001 C CNN "LCSC"
+	1    9900 5950
+	0    1    1    0
+$EndComp
+Wire Wire Line
+	9000 5950 9550 5950
 Wire Wire Line
 	9000 6850 9700 6850
@@
 L Device:R R23
 U 1 1 60F2A22E
-P 9850 6150
-F 0 "R23" V 9800 6350 50  0000 C CNN
-F 1 "10K" V 9900 5950 50  0000 C CNN
-F 2 "Resistor_SMD:R_0603_1608Metric" V 9780 6150 50  0001 C CNN
-F 3 "~" H 9850 6150 50  0001 C CNN
-F 4 "C98220" V 9850 6150 50  0001 C CNN "LCSC"
-	1    9850 6150
-	0    1    1    0
-$EndComp
-Wire Wire Line
-	9000 6150 9700 6150
+P 9900 6150
+F 0 "R23" V 9850 6350 50  0000 C CNN
+F 1 "10K" V 9950 5950 50  0000 C CNN
+F 2 "Resistor_SMD:R_0603_1608Metric" V 9830 6150 50  0001 C CNN
+F 3 "~" H 9900 6150 50  0001 C CNN
+F 4 "C98220" V 9900 6150 50  0001 C CNN "LCSC"
+	1    9900 6150
+	0    1    1    0
+$EndComp
+Wire Wire Line
+	9000 6150 9750 6150
 $Comp
 L power:+3.3VP #PWR0126
 U 1 1 60F44A4B
-P 10600 5950
-F 0 "#PWR0126" H 10750 5900 50  0001 C CNN
-F 1 "+3.3VP" V 10615 6078 50  0000 L CNN
-F 2 "" H 10600 5950 50  0001 C CNN
-F 3 "" H 10600 5950 50  0001 C CNN
-	1    10600 5950
-	0    1    1    0
-$EndComp
-Wire Wire Line
-	10000 5950 10250 5950
-Wire Wire Line
-	10600 6150 10600 5950
-Wire Wire Line
-	10000 6150 10600 6150
-Connection ~ 10600 5950
-Wire Wire Line
-	10250 6650 10250 6850
+P 10250 5950
+F 0 "#PWR0126" H 10400 5900 50  0001 C CNN
+F 1 "+3.3VP" V 10265 6078 50  0000 L CNN
+F 2 "" H 10250 5950 50  0001 C CNN
+F 3 "" H 10250 5950 50  0001 C CNN
+	1    10250 5950
+	0    1    1    0
+$EndComp
 Wire Wire Line
 	10000 6850 10250 6850
-Wire Wire Line
-	10250 6250 10250 5950
-Connection ~ 10250 5950
-Wire Wire Line
-	10250 5950 10600 5950
 Wire Wire Line
 	10250 6850 10250 7250
@@
 L Device:R R8
 U 1 1 6135F07C
-P 5000 6500
-F 0 "R8" V 4950 6700 50  0000 C CNN
-F 1 "2.2K" V 5050 6300 50  0000 C CNN
-F 2 "Resistor_SMD:R_0603_1608Metric" V 4930 6500 50  0001 C CNN
-F 3 "~" H 5000 6500 50  0001 C CNN
-F 4 "C25992" V 5000 6500 50  0001 C CNN "LCSC"
-	1    5000 6500
-	0    1    1    0
-$EndComp
-$Comp
-L Device:R R7
-U 1 1 6137CF15
 P 5000 6400
-F 0 "R7" V 4950 6600 50  0000 C CNN
+F 0 "R8" V 4950 6600 50  0000 C CNN
 F 1 "2.2K" V 5050 6200 50  0000 C CNN
 F 2 "Resistor_SMD:R_0603_1608Metric" V 4930 6400 50  0001 C CNN
@@
 	0    1    1    0
 $EndComp
-Wire Wire Line
-	4550 6400 4850 6400
-Wire Wire Line
-	4550 6500 4850 6500
+$Comp
+L Device:R R7
+U 1 1 6137CF15
+P 5000 6300
+F 0 "R7" V 4950 6500 50  0000 C CNN
+F 1 "2.2K" V 5050 6100 50  0000 C CNN
+F 2 "Resistor_SMD:R_0603_1608Metric" V 4930 6300 50  0001 C CNN
+F 3 "~" H 5000 6300 50  0001 C CNN
+F 4 "C25992" V 5000 6300 50  0001 C CNN "LCSC"
+	1    5000 6300
+	0    1    1    0
+$EndComp
 $Comp
 L Device:LED_Small_ALT D8
 U 1 1 613BD51C
-P 5400 6300
-F 0 "D8" V 5400 6230 50  0000 R CNN
-F 1 "LED_Small_ALT" V 5355 6230 50  0001 R CNN
-F 2 "Diode_SMD:D_0603_1608Metric" V 5400 6300 50  0001 C CNN
-F 3 "~" V 5400 6300 50  0001 C CNN
-F 4 "C72043" V 5400 6300 50  0001 C CNN "LCSC"
-	1    5400 6300
-	0    -1   -1   0
-$EndComp
-Wire Wire Line
-	5150 6400 5400 6400
-Wire Wire Line
-	5150 6500 5750 6500
-Wire Wire Line
-	5750 6500 5750 6400
+P 5400 6200
+F 0 "D8" V 5400 6130 50  0000 R CNN
+F 1 "LED_Small_ALT" V 5355 6130 50  0001 R CNN
+F 2 "Diode_SMD:D_0603_1608Metric" V 5400 6200 50  0001 C CNN
+F 3 "~" V 5400 6200 50  0001 C CNN
+F 4 "C72043" V 5400 6200 50  0001 C CNN "LCSC"
+	1    5400 6200
+	0    -1   -1   0
+$EndComp
+Wire Wire Line
+	5150 6300 5400 6300
+Wire Wire Line
+	5150 6400 5750 6400
+Wire Wire Line
+	5750 6400 5750 6300
 $Comp
 L power:+3.3V #PWR0132
 U 1 1 6142CBFA
-P 5400 6200
-F 0 "#PWR0132" H 5400 6050 50  0001 C CNN
-F 1 "+3.3V" H 5415 6373 50  0000 C CNN
-F 2 "" H 5400 6200 50  0001 C CNN
-F 3 "" H 5400 6200 50  0001 C CNN
-	1    5400 6200
-	1    0    0    -1
-$EndComp
-Wire Wire Line
-	5400 6200 5750 6200
-Connection ~ 5400 6200
+P 5400 6100
+F 0 "#PWR0132" H 5400 5950 50  0001 C CNN
+F 1 "+3.3V" H 5415 6273 50  0000 C CNN
+F 2 "" H 5400 6100 50  0001 C CNN
+F 3 "" H 5400 6100 50  0001 C CNN
+	1    5400 6100
+	1    0    0    -1
+$EndComp
+Wire Wire Line
+	5400 6100 5750 6100
+Connection ~ 5400 6100
 $Comp
 L Device:LED_Small_ALT D9
 U 1 1 61450534
-P 5750 6300
-F 0 "D9" V 5750 6230 50  0000 R CNN
-F 1 "LED_Small_ALT" V 5705 6230 50  0001 R CNN
-F 2 "Diode_SMD:D_0603_1608Metric" V 5750 6300 50  0001 C CNN
-F 3 "~" V 5750 6300 50  0001 C CNN
-F 4 "C72043" V 5750 6300 50  0001 C CNN "LCSC"
-	1    5750 6300
+P 5750 6200
+F 0 "D9" V 5750 6130 50  0000 R CNN
+F 1 "LED_Small_ALT" V 5705 6130 50  0001 R CNN
+F 2 "Diode_SMD:D_0603_1608Metric" V 5750 6200 50  0001 C CNN
+F 3 "~" V 5750 6200 50  0001 C CNN
+F 4 "C72043" V 5750 6200 50  0001 C CNN "LCSC"
+	1    5750 6200
 	0    -1   -1   0
 $EndComp
@@
 NoConn ~ 4550 6000
 NoConn ~ 4550 6100
-NoConn ~ 4550 6300
 NoConn ~ 4550 7100
 NoConn ~ 4550 7200
@@
 Wire Wire Line
 	8500 1400 8550 1400
+Wire Wire Line
+	4550 6300 4850 6300
+Wire Wire Line
+	4550 6400 4850 6400
+NoConn ~ 4550 6500
+Wire Wire Line
+	10250 6600 10250 6850
+Wire Wire Line
+	9550 6600 9550 5950
+Connection ~ 9550 5950
+Wire Wire Line
+	9550 5950 9750 5950
+Wire Wire Line
+	9550 6600 9700 6600
+Wire Wire Line
+	10100 6600 10250 6600
+Wire Wire Line
+	10050 5950 10250 5950
+Wire Wire Line
+	10050 6150 10250 6150
+Wire Wire Line
+	10250 6150 10250 5950
+Connection ~ 10250 5950
 $EndSCHEMATC

Commit message: done
Parts:
- removed D7: 2V7, Package_TO_SOT_SMD:SOT-223, symbol Device:D_Zener
- removed J3: Conn_01x06, Connector_PinHeader_2.54mm:PinHeader_1x06_P2.54mm_Vertical, symbol Connector_Generic:Conn_01x06
- added D7: 2V7, Package_TO_SOT_SMD:SOT-223, symbol HKIA_Tracker_SYM:D_Zener_BZV90
- added H1, H2: M3, MountingHole:MountingHole_3.2mm_M3_Pad, symbol Mechanical:MountingHole
- added J3: NFC_ANT, Connector_PinHeader_2.54mm:PinHeader_1x02_P2.54mm_Vertical, symbol Connector_Generic:Conn_01x02
- J1: footprint Connector_PinHeader_2.54mm:PinHeader_1x03_P2.54mm_Horizontal -> Connector_PinHeader_2.54mm:PinHeader_1x03_P2.54mm_Vertical
Connections:
- net labels removed: GPIO12, GPIO13, GPIO14, GPIO15
- wire segments 249 -> 237
- no-connect marks 28 -> 32
Other:
- note removed: "ANT"
Changed lines of the file:
@@
 U 1 1 60A5B54F
 P 1250 1600
-F 0 "J1" H 1168 1917 50  0000 C CNN
-F 1 "Motor In" H 1168 1826 50  0000 C CNN
-F 2 "Connector_PinHeader_2.54mm:PinHeader_1x03_P2.54mm_Horizontal" H 1250 1600 50  0001 C CNN
+F 0 "J1" H 1168 1275 50  0000 C CNN
+F 1 "Motor In" H 1168 1366 50  0000 C CNN
+F 2 "Connector_PinHeader_2.54mm:PinHeader_1x03_P2.54mm_Vertical" H 1250 1600 50  0001 C CNN
 F 3 "~" H 1250 1600 50  0001 C CNN
 	1    1250 1600
-	-1   0    0    -1
+	-1   0    0    1
 $EndComp
 Wire Wire Line
@@
 	1    3850 1650
 	1    0    0    -1
-$EndComp
-$Comp
-L Device:D_Zener D7
-U 1 1 60A604E8
-P 3000 1650
-F 0 "D7" V 2954 1730 50  0000 L CNN
-F 1 "2V7" V 3045 1730 50  0000 L CNN
-F 2 "Package_TO_SOT_SMD:SOT-223" H 3000 1650 50  0001 C CNN
-F 3 "https://assets.nexperia.com/documents/data-sheet/BZV90.pdf" H 3000 1650 50  0001 C CNN
-F 4 "1727-5570-1-ND" V 3000 1650 50  0001 C CNN "DIGI"
-	1    3000 1650
-	0    1    1    0
 $EndComp
 Wire Wire Line
@@
 Wire Wire Line
 	4550 6200 4900 6200
-Wire Wire Line
-	5000 5300 5000 5400
-Wire Notes Line
-	4800 5450 5100 5450
-Wire Notes Line
-	5100 5450 5100 5250
-Wire Notes Line
-	5100 5250 4800 5250
-Wire Notes Line
-	4800 5250 4800 5450
-Text Notes 5150 5450 0    50   ~ 0
-ANT
 $Comp
 L power:+BATT #PWR0128
@@
 	0    -1   -1   0
 $EndComp
-Text Label 4700 5600 0    50   ~ 0
-GPIO12
-Wire Wire Line
-	4550 5600 5000 5600
-Text Label 4700 5700 0    50   ~ 0
-GPIO13
-Wire Wire Line
-	4550 5700 5000 5700
-Text Label 4700 5800 0    50   ~ 0
-GPIO14
-Wire Wire Line
-	4550 5800 5000 5800
-Text Label 4700 5900 0    50   ~ 0
-GPIO15
-Wire Wire Line
-	4550 5900 5000 5900
 $Comp
 L Switch:SW_Push SW2
@@
 	0    -1   -1   0
 $EndComp
-Wire Wire Line
-	8100 4500 8600 4500
-$Comp
-L power:+3.3V #PWR0133
-U 1 1 612F56ED
-P 8600 4500
-F 0 "#PWR0133" H 8600 4350 50  0001 C CNN
-F 1 "+3.3V" V 8615 4628 50  0000 L CNN
-F 2 "" H 8600 4500 50  0001 C CNN
-F 3 "" H 8600 4500 50  0001 C CNN
-	1    8600 4500
-	0    1    1    0
-$EndComp
-Wire Wire Line
-	8150 5000 8150 5050
-Wire Wire Line
-	8100 5000 8150 5000
-$Comp
-L power:GND #PWR0134
-U 1 1 612E58D3
-P 8150 5050
-F 0 "#PWR0134" H 8150 4800 50  0001 C CNN
-F 1 "GND" H 8155 4877 50  0000 C CNN
-F 2 "" H 8150 5050 50  0001 C CNN
-F 3 "" H 8150 5050 50  0001 C CNN
-	1    8150 5050
-	1    0    0    -1
-$EndComp
-$Comp
-L Connector_Generic:Conn_01x06 J3
-U 1 1 612E3F7A
-P 7900 4700
-F 0 "J3" H 7818 5117 50  0000 C CNN
-F 1 "Conn_01x06" H 7818 5026 50  0000 C CNN
-F 2 "Connector_PinHeader_2.54mm:PinHeader_1x06_P2.54mm_Vertical" H 7900 4700 50  0001 C CNN
-F 3 "~" H 7900 4700 50  0001 C CNN
-	1    7900 4700
-	-1   0    0    -1
-$EndComp
-Wire Wire Line
-	8100 4900 8550 4900
-Text Label 8250 4900 0    50   ~ 0
-GPIO15
-Wire Wire Line
-	8100 4800 8550 4800
-Text Label 8250 4800 0    50   ~ 0
-GPIO14
-Wire Wire Line
-	8100 4700 8550 4700
-Text Label 8250 4700 0    50   ~ 0
-GPIO13
-Wire Wire Line
-	8100 4600 8550 4600
-Text Label 8250 4600 0    50   ~ 0
-GPIO12
 Connection ~ 12200 5100
 $Comp
@@
 	10250 6150 10250 5950
 Connection ~ 10250 5950
+$Comp
+L HKIA_Tracker_SYM:D_Zener_BZV90 D7
+U 1 1 61B18AB6
+P 3000 1650
+F 0 "D7" V 2954 1730 50  0000 L CNN
+F 1 "2V7" V 3045 1730 50  0000 L CNN
+F 2 "Package_TO_SOT_SMD:SOT-223" H 3050 1750 50  0001 C CNN
+F 3 "~" H 3000 1650 50  0001 C CNN
+F 4 "1727-5570-1-ND" V 3000 1650 50  0001 C CNN "DIGI"
+	1    3000 1650
+	0    1    1    0
+$EndComp
+$Comp
+L Mechanical:MountingHole H1
+U 1 1 61B451E0
+P 13750 2100
+F 0 "H1" H 13850 2146 50  0000 L CNN
+F 1 "M3" H 13850 2055 50  0000 L CNN
+F 2 "MountingHole:MountingHole_3.2mm_M3_Pad" H 13750 2100 50  0001 C CNN
+F 3 "~" H 13750 2100 50  0001 C CNN
+	1    13750 2100
+	1    0    0    -1
+$EndComp
+$Comp
+L Mechanical:MountingHole H2
+U 1 1 61B46062
+P 13750 2350
+F 0 "H2" H 13850 2396 50  0000 L CNN
+F 1 "M3" H 13850 2305 50  0000 L CNN
+F 2 "MountingHole:MountingHole_3.2mm_M3_Pad" H 13750 2350 50  0001 C CNN
+F 3 "~" H 13750 2350 50  0001 C CNN
+	1    13750 2350
+	1    0    0    -1
+$EndComp
+NoConn ~ 4550 5600
+NoConn ~ 4550 5700
+NoConn ~ 4550 5800
+NoConn ~ 4550 5900
+$Comp
+L Connector_Generic:Conn_01x02 J3
+U 1 1 61C670EC
+P 5200 5300
+F 0 "J3" H 5280 5292 50  0000 L CNN
+F 1 "NFC_ANT" H 5280 5201 50  0000 L CNN
+F 2 "Connector_PinHeader_2.54mm:PinHeader_1x02_P2.54mm_Vertical" H 5200 5300 50  0001 C CNN
+F 3 "~" H 5200 5300 50  0001 C CNN
+	1    5200 5300
+	1    0    0    -1
+$EndComp
 $EndSCHEMATC
